Commit message: v1.0.1

File: source/robot_lab/data/Robots/TSD/TSD2/urdf/TSD2.urdf (robot description, URDF)
Before this commit: robot TSD2, 17 links, 16 joints
Joints:
- joint FL_calf_joint: limit lower=-2.7576 upper=2.5831 effort=170.0 velocity=180.0 -> lower=-2.7576 upper=2.5831 effort=170.0 velocity=18.84955592153876
- joint FL_hip_joint: limit lower=-0.61087 upper=0.43633 effort=170.0 velocity=180.0 -> lower=-0.61087 upper=0.43633 effort=170.0 velocity=18.84955592153876
- joint FL_thigh_joint: limit lower=-2.4435 upper=2.4435 effort=170.0 velocity=180.0 -> lower=-2.4435 upper=2.4435 effort=170.0 velocity=18.84955592153876
- joint FL_wheel_joint: limit lower=0.0 upper=0.0 effort=38.0 velocity=590.0 -> effort=38.0 velocity=61.784655520599266
- joint FR_calf_joint: limit lower=-2.7576 upper=2.5831 effort=170.0 velocity=180.0 -> lower=-2.7576 upper=2.5831 effort=170.0 velocity=18.84955592153876
- joint FR_hip_joint: limit lower=-0.61087 upper=0.43633 effort=170.0 velocity=180.0 -> lower=-0.61087 upper=0.43633 effort=170.0 velocity=18.84955592153876
- joint FR_thigh_joint: limit lower=-2.4435 upper=2.4435 effort=170.0 velocity=180.0 -> lower=-2.4435 upper=2.4435 effort=170.0 velocity=18.84955592153876
- joint FR_wheel_joint: limit lower=0.0 upper=0.0 effort=38.0 velocity=590.0 -> effort=38.0 velocity=61.784655520599266
- joint RL_calf_joint: limit lower=-2.7576 upper=2.5831 effort=170.0 velocity=180.0 -> lower=-2.7576 upper=2.5831 effort=170.0 velocity=18.84955592153876
- joint RL_hip_joint: limit lower=-0.61087 upper=0.43633 effort=170.0 velocity=180.0 -> lower=-0.61087 upper=0.43633 effort=170.0 velocity=18.84955592153876
- joint RL_thigh_joint: limit lower=-2.4435 upper=2.4435 effort=170.0 velocity=180.0 -> lower=-2.4435 upper=2.4435 effort=170.0 velocity=18.84955592153876
- joint RL_wheel_joint: limit lower=0.0 upper=0.0 effort=38 velocity=590.0 -> effort=38 velocity=61.784655520599266
- joint RR_calf_joint: limit lower=-2.7576 upper=2.5831 effort=170.0 velocity=180.0 -> lower=-2.7576 upper=2.5831 effort=170.0 velocity=18.84955592153876
- joint RR_hip_joint: limit lower=-0.61087 upper=0.43633 effort=170.0 velocity=180.0 -> lower=-0.61087 upper=0.43633 effort=170.0 velocity=18.84955592153876
- joint RR_thigh_joint: limit lower=-2.4435 upper=2.4435 effort=170.0 velocity=180.0 -> lower=-2.4435 upper=2.4435 effort=170.0 velocity=18.84955592153876
- joint RR_wheel_joint: limit lower=0.0 upper=0.0 effort=38.0 velocity=590.0 -> effort=38.0 velocity=61.784655520599266

Commit message: v1.0.1

File: source/robot_lab/data/Robots/TSD/TSD2/urdf/TSD2.urdf (robot description, URDF)
Before this commit: robot TSD2, 17 links, 16 joints
Links:
- link FL_calf: mass 1.1494 -> 1.09119252955386
- link FL_hip: mass 0.88356 -> 0.894912703451862
- link FL_thigh: mass 1.045 -> 1.06633586725301
- link FL_wheel: mass 1.3002 -> 0.809759882175001
- link FR_calf: mass 1.1494 -> 1.0911925295716
- link FR_hip: mass 0.88356 -> 0.89491
- link FR_thigh: mass 1.045 -> 1.0663
- link FR_wheel: mass 1.3002 -> 0.80976
- link RL_calf: mass 1.1494 -> 1.09119252958064
- link RL_hip: mass 0.88356 -> 0
- link RL_thigh: mass 1.045 -> 1.06633596148158
- link RL_wheel: mass 1.3002 -> 0.809759882175001
- link RR_calf: mass 1.1046 -> 1.09119252957151
- link RR_hip: mass 0.88356 -> 0.894912736354396
- link RR_thigh: mass 1.045 -> 1.06633596228652
- link RR_wheel: mass 1.3002 -> 0.809759882174997
- link base_link: mass 16.936 -> 19
Joints:
- joint FL_calf_joint: limit lower=-2.7576 upper=2.5831 effort=170.0 velocity=18.84955592153876 -> lower=-2.7576 upper=2.5831 effort=170 velocity=18.8495559215388
- joint FL_hip_joint: limit lower=-0.61087 upper=0.43633 effort=170.0 velocity=18.84955592153876 -> lower=-0.61087 upper=0.43633 effort=170 velocity=18.8495559215388
- joint FL_thigh_joint: limit lower=-2.4435 upper=2.4435 effort=170.0 velocity=18.84955592153876 -> lower=-2.4435 upper=2.4435 effort=170 velocity=18.8495559215388
- joint FL_wheel_joint: limit effort=38.0 velocity=61.784655520599266 -> lower=0 upper=0 effort=38 velocity=61.7846555205993
- joint FR_calf_joint: limit lower=-2.7576 upper=2.5831 effort=170.0 velocity=18.84955592153876 -> lower=-2.7576 upper=2.5831 effort=170 velocity=18.85
- joint FR_hip_joint: limit lower=-0.61087 upper=0.43633 effort=170.0 velocity=18.84955592153876 -> lower=-0.61087 upper=0.43633 effort=170 velocity=18.85
- joint FR_thigh_joint: limit lower=-2.4435 upper=2.4435 effort=170.0 velocity=18.84955592153876 -> lower=-2.4435 upper=2.4435 effort=170 velocity=18.85
- joint FR_wheel_joint: limit effort=38.0 velocity=61.784655520599266 -> lower=0 upper=0 effort=38 velocity=61.7846555205993
- joint RL_calf_joint: limit lower=-2.7576 upper=2.5831 effort=170.0 velocity=18.84955592153876 -> lower=-2.7576 upper=2.5831 effort=170 velocity=18.85
- joint RL_hip_joint: limit lower=-0.61087 upper=0.43633 effort=170.0 velocity=18.84955592153876 -> lower=-0.61087 upper=0.43633 effort=170 velocity=18.85
- joint RL_thigh_joint: limit lower=-2.4435 upper=2.4435 effort=170.0 velocity=18.84955592153876 -> lower=-2.4435 upper=2.4435 effort=170 velocity=18.8495559215388
- joint RL_wheel_joint: limit effort=38 velocity=61.784655520599266 -> lower=0 upper=0 effort=38 velocity=61.785
- joint RR_calf_joint: limit lower=-2.7576 upper=2.5831 effort=170.0 velocity=18.84955592153876 -> lower=-2.7576 upper=2.5831 effort=170 velocity=18.8495559215388
- joint RR_hip_joint: limit lower=-0.61087 upper=0.43633 effort=170.0 velocity=18.84955592153876 -> lower=-0.61087 upper=0.43633 effort=170 velocity=18.8495559215388
- joint RR_thigh_joint: limit lower=-2.4435 upper=2.4435 effort=170.0 velocity=18.84955592153876 -> lower=-2.4435 upper=2.4435 effort=170 velocity=18.8495559215388
- joint RR_wheel_joint: limit effort=38.0 velocity=61.784655520599266 -> lower=0 upper=0 effort=38 velocity=61.785

Commit message: v1.0.1

File: source/robot_lab/data/Robots/TSD/TSD2/urdf/TSD2.urdf (robot description, URDF)
Before this commit: robot TSD2, 17 links, 16 joints
Joints:
- joint FL_wheel_joint: limit lower=0 upper=0 effort=38 velocity=61.7846555205993 -> effort=38 velocity=61.7846555205993
- joint FR_wheel_joint: limit lower=0 upper=0 effort=38 velocity=61.7846555205993 -> effort=38 velocity=61.7846555205993
- joint RL_wheel_joint: limit lower=0 upper=0 effort=38 velocity=61.785 -> effort=38 velocity=61.785
- joint RR_wheel_joint: limit lower=0 upper=0 effort=38 velocity=61.785 -> effort=38 velocity=61.785

Commit message: v1.0.1

File: source/robot_lab/data/Robots/TSD/TSD2/urdf/TSD2.urdf (robot description, URDF)
Before this commit: robot TSD2, 17 links, 16 joints
Links:
- link RL_hip: mass 0 -> 0.88356
